File: digi_analog_clock.sch (KiCad schematic (older format))
At the start: 20 parts

Commit message: Add sk6805 blocks
Parts:
- removed R?: 10kR, symbol Device:R
- removed R?: 20kR, symbol Device:R
- removed U?: IS31FL3731, symbol Driver_LED:IS31FL3731
- added R3: 600R, Resistor_SMD:R_0805_2012Metric, symbol Device:R
- BT1: renamed from BT?; footprint (none) -> Battery:BatteryHolder_Keystone_3034_1x20mm
- C1, C2, C3, C4: renamed from C?; footprint (none) -> Capacitor_SMD:C_0805_2012Metric
- R1, R2, R4, R5, R6, R7, R8: renamed from R?; footprint (none) -> Resistor_SMD:R_0805_2012Metric
- SW1, SW2: renamed from SW?; footprint (none) -> Button_Switch_SMD:SW_SPST_CK_RS282G05A3
- U2: renamed from U?; footprint (none) -> Package_SO:SOIC-8-1EP_3.9x4.9mm_P1.27mm_EP2.29x3mm
- Y1: renamed from Y?; footprint (none) -> Crystal:Crystal_SMD_G8-2Pin_3.2x1.5mm
- gave numbers to parts that had none: 1
Connections:
- net labels added: SCL, SDA
- wire segments 85 -> 164
- no-connect marks 4 -> 1

Commit message: Some updates, not finished
Parts:
- added J1: USB_B_Micro, digikey-footprints:USB_Micro_B_Female_10118194-0001LF, symbol Connector:USB_B_Micro
Connections:
- net +5V: now also J1.1 (VBUS)
- net GND: now also J1.5 (GND), J1.6 (Shield)
- no-connect marks 1 -> 4

Commit message: Use atsamd21; do most layout
Parts:
- removed R8: 10kR, Resistor_SMD:R_0805_2012Metric, symbol Device:R
- removed U1: ATtiny13A-SSU, Package_SO:SOIC-8_3.9x4.9mm_P1.27mm, symbol MCU_Microchip_ATtiny:ATtiny13A-SSU
- added C1, C2: 1uF, Capacitor_SMD:C_0805_2012Metric, symbol Device:C
- added C5: 10kpF, Capacitor_SMD:C_0603_1608Metric, symbol Device:C_Small
- added C6, C7, C8: 10kpF, Capacitor_SMD:C_0603_1608Metric, symbol Device:C
- added J2: Conn_ARM_JTAG_SWD_10, Connector_PinHeader_1.27mm:PinHeader_2x05_P1.27mm_Vertical_SMD, symbol Connector:Conn_ARM_JTAG_SWD_10
- added R10, R12, R14, R16: 10kR, Resistor_SMD:R_0805_2012Metric, symbol Device:R
- added R11, R13, R15, R9: 1kR, Resistor_SMD:R_0805_2012Metric, symbol Device:R
- added R8: 10kR, Resistor_SMD:R_0805_2012Metric, symbol Device:R_Small
- added SW1, SW2: SW_Push, WM_lib:SW_Push_1P1T_Vertical_CK_PTS815, symbol Switch:SW_Push
- added U2: TC2014-3.3VxCTTR, Package_TO_SOT_SMD:SOT-23-5, symbol Regulator_Linear:TC2014-3.3VxCTTR
- added U3: ATSAMD21E15L-A, Package_QFP:TQFP-32_7x7mm_P0.8mm, symbol MCU_Microchip_SAMD:ATSAMD21E15L-A
- added U4: ATtiny10-TS, Package_TO_SOT_SMD:SOT-23-6, symbol MCU_Microchip_ATtiny:ATtiny10-TS
- C10: renamed from C2; value 1uF -> 10kpF; footprint Capacitor_SMD:C_0805_2012Metric -> Capacitor_SMD:C_0603_1608Metric
- C9: renamed from C1; value 1uF -> 10kpF; footprint Capacitor_SMD:C_0805_2012Metric -> Capacitor_SMD:C_0603_1608Metric
- R3: value 600R -> 10kR
- SW3: renamed from SW1; footprint Button_Switch_SMD:SW_SPST_CK_RS282G05A3 -> WM_lib:SW_Push_1P1T_Vertical_CK_PTS815
- SW4: renamed from SW2; footprint Button_Switch_SMD:SW_SPST_CK_RS282G05A3 -> WM_lib:SW_Push_1P1T_Vertical_CK_PTS815
- U1: renamed from U2; footprint Package_SO:SOIC-8-1EP_3.9x4.9mm_P1.27mm_EP2.29x3mm -> Package_SO:SOIC-8_3.9x4.9mm_P1.27mm
Connections:
- net 6x_sk6805_1515_mins_1/DIN is gone; now on net +3.3V: R3.1
- net +5V: now also C1.1, R8.1, U2.1 (VIN), U4.5 (VCC); no longer R1.2, R2.2, R6.1, U1.8 (VCC)
- net GND: now also C10.1, C9.1, J1.2 (D-), J1.3 (D+), J1.4 (ID), SW3.2, SW4.2, C1.2, C2.2, C5.2, C6.1, C7.1, C8.1, J2.3 (GND), J2.5 (GND), J2.9 (GNDDetect), SW1.2, SW2.2, U2.2 (GND), U3.10 (GND), U3.26 (GND), U4.2 (GND); no longer C10.2, C9.2, SW3.1, SW4.1
- net SCL: now also R3.2, U3.22 (PA23); no longer R1.1
- net SDA: now also R4.2, U3.21 (PA22); no longer R2.1
- net SWDIO: now reaches R6.2
- net SWDIO: now also J2.2 (SWDIO/TMS), U3.30 (PA31)
- net SWDCLK: now reaches R5.2
- net SWDCLK: now also J2.4 (SWDCLK/TCK), U3.29 (PA30); no longer C10.1
- net MFP: now reaches U1.7 (MFP)
- net MFP: now also R2.2, U3.7 (PA06)
- net +3.3V: now reaches R5.1
- net +3.3V: now also R1.1, R2.1, R4.1, R6.1, U1.8 (VCC), C2.1, J2.1 (VTref), R10.1, R12.1, R14.1, R16.1, U2.5 (VOUT), U3.28 (VDDIO), U3.9 (VDDIO/VDDANA); no longer SW4.2
- new net: R15.1, SW4.1
- new net: R13.1, SW3.1
- new net: R11.1, SW2.1
- new net: C6.2, U3.27 (VDDCORE)
- new net: R8.2, U2.3 (ON/~OFF~)
- new net: C5.1, U2.4 (BP)
- new net: R9.1, SW1.1
- new net HH: C9.2, R13.2, R14.2, U3.2 (PA03)
- new net LED: U4.4 (PB2)
- new net MM: C10.2, R15.2, R16.2, U3.1 (PA02)
- new net MODE1: C8.2, R11.2, R12.2, U3.5 (PA04)
- new net MODE2: C7.2, R10.2, R9.2, U3.6 (PA05)
- new net MOSI: U3.17 (PA16), U4.3 (PB1)
- new net RESET3.3: J2.10 (~RESET~), R1.2, U3.25 (~RESET)
- new net RESET5: R7.2, U4.6 (~RESET~/PB3)
- new net SCK: U3.18 (PA17), U4.1 (PB0)
- no-connect marks 4 -> 18
Other:
- note added: "3.3V LDO"
- note added: "RTC"
- note added: "SERCOM1"
- note added: "SERCOM3"
- note added: "SPI -> WS2812"
- moved on the sheet: BT1, C10, C3, C4, C9, SW3, SW4, U1, Y1
